File: Swicher.sch (KiCad schematic (older format))
At the start: 61 parts, among them K1 RELAY, P1 CONN_01X02, P10 CONN_01X04, P11 CONN_01X04, P12 CONN_01X04, P13 CONN_01X04, P2 CONN_01X02, P3 CONN_01X04, P4 CONN_01X04, P5 CONN_01X04, P6 CONN_01X02, P7 CONN_01X04, P8 CONN_01X04, P9 BDM, Q1 BC237, SW1 RESET, SW2 SP3T, T1 TRANSFO, U1 MC9S08SH8, U10 4N25, U11 4N25, U12 4N25, U13 4N25, U14 4N25, U2 78L05, U3 4N25, U4 4N25, U5 4N25, U6 4N25, U7 4N25, U8 4N25, U9 4N25

Commit message: cambio relay
Parts:
- K1: footprint Relays_ThroughHole:Relay_SANYOU_SRD_Series_Form_C -> locales:RELAY-HJQ-15F
Changed lines of the file:
@@
 F 0 "K1" H 8285 4355 70  0000 C CNN
 F 1 "RELAY" H 8185 3855 70  0000 C CNN
-F 2 "Relays_ThroughHole:Relay_SANYOU_SRD_Series_Form_C" H 8035 4355 60  0001 C CNN
+F 2 "locales:RELAY-HJQ-15F" H 8035 4355 60  0001 C CNN
 F 3 "" H 8035 4355 60  0000 C CNN
 	1    8035 4355
